File: hardware/NCS199A3R_test/NCS199A3R_test.kicad_sch (KiCad schematic)
At the start: 11 parts, among them U1 NCS199A3RSQT2G

Commit message: panelization
Other:
- note added: "Let's say we want to measure from -3.5A to 3.5A We want that to be between 0V to 3.3V 0A means 3.3/2 = 1.65V (cf REF voltage) R=U/I ; Umax = 1.65 / 200 = 0.00825V R = 0.00825 / 3.5 = 0.0023R"
Changed lines of the file:
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@@
     (stroke (width 0) (type default) (color 0 0 0 0))
+  )
+  (text "Let's say we want to measure from -3.5A to 3.5A\nWe want that to be between 0V to 3.3V\n0A means 3.3/2 = 1.65V (cf REF voltage)\nR=U/I ; Umax = 1.65 / 200 = 0.00825V\nR = 0.00825 / 3.5 = 0.0023R"
+    (at 44.45 81.28 0)
+    (effects (font (size 1.27 1.27)) (justify left bottom))
   )
   (text "Gain = 200" (at 127 88.9 0)
