File: hardware/gc_STM32G491CET6/gc_STM32G491CET6.kicad_sch (KiCad schematic)
At the start: 4 parts

Commit message: Schematics + rough placement
Parts:
- H101, H102, H103, H104: renamed from H?; value MountingHole_Pad -> MountingHole_3.2mm_M3_Pad_Via
Other:
- sheet Actuators ports: added M1_ADC_ISENSE, M1_ENC_A, M1_ENC_B, M1_TIM_FWD, M1_TIM_REV, M2_ADC_ISENSE, M2_ENC_A, M2_ENC_B, M2_TIM_FWD, M2_TIM_REV, XL320_UART; removed none
- sheet Power Supply ports: added BAT_SENSE, USB_DM, USB_DP; removed none
- sheet Sensors ports: added FLOOR_1, FLOOR_2, TCS3200_LED, TCS3200_S2, TCS3200_S3, TCS3200_TIM, TOF1_GPIO1, TOF1_XSHUT, TOF2_GPIO1, TOF2_XSHUT, TOF_I2C_SCL, TOF_I2C_SDA; removed none
- moved on the sheet: H101, H102, H103, H104

Commit message: started routing
Other:
- sheet Power Supply ports: added USB_DN; removed USB_DM
- sheet STM32 ports: added USB_DN; removed USB_DM
Changed lines of the file:
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@@
       (effects (font (size 1.27 1.27)) (justify right))
     )
-    (pin "USB_DM" input (at 127 105.41 90)
+    (pin "USB_DN" input (at 127 105.41 90)
       (effects (font (size 1.27 1.27)) (justify right))
     )
@@
       (effects (font (size 1.27 1.27)) (justify right))
     )
-    (pin "USB_DM" input (at 127 88.9 270)
+    (pin "USB_DN" input (at 127 88.9 270)
       (effects (font (size 1.27 1.27)) (justify left))
     )
