File: hardware/gc_STM32G491CET6/sensors.kicad_sch (KiCad schematic)
At the start: 5 parts

Commit message: Schematics + rough placement
Parts:
- removed J?: COLOR, Connector_JST:JST_XH_B4B-XH-A_1x04_P2.50mm_Vertical, symbol Connector_Generic:Conn_01x04
- added J505: TCS3200, Connector_JST:JST_XH_B6B-XH-A_1x06_P2.50mm_Vertical, symbol Connector_Generic:Conn_01x06
- added R501, R502: 2.2k, Resistor_SMD:R_0603_1608Metric, symbol Device:R_Small
- J501: renamed from J?; value TOF -> TOF1
- J502: renamed from J?; value TOF -> TOF2
- gave numbers to parts that had none: 2
Connections:
- net GND: now also J505.6 (Pin_6)
- net +3V3 renamed +3.3V
- net +3.3V: now also J505.1 (Pin_1), R501.1, R502.1
- net FLOOR_SENSOR1 renamed FLOOR_1
- net FLOOR_SENSOR2 renamed FLOOR_2
- net I2C_TOF_SCL renamed TOF_I2C_SCL
- net TOF_I2C_SCL: now also R502.2
- net I2C_TOF_SDA renamed TOF_I2C_SDA
- net TOF_I2C_SDA: now also R501.2
- net TOF_GPIO1 renamed TOF1_GPIO1
- net TOF1_GPIO1: no longer J502.6 (Pin_6)
- net TOF_XSHUT renamed TOF1_XSHUT
- net TOF1_XSHUT: no longer J502.5 (Pin_5)
- new net TCS3200_LED: J505.3 (Pin_3)
- new net TCS3200_S2: J505.5 (Pin_5)
- new net TCS3200_S3: J505.4 (Pin_4)
- new net TCS3200_TIM: J505.2 (Pin_2)
- new net TOF2_GPIO1: J502.6 (Pin_6)
- new net TOF2_XSHUT: J502.5 (Pin_5)
Other:
- note added: "I2C pull-up resistors Do not fit, already present on pololu's board"
- note added: "TCS3200 Color sensor connector"
- note removed: "Connector for color sensor"
- moved on the sheet: J501, J502, J503, J504
